Commit message: Assignment 1 - Add a can to the robot

File: src/bumperbot_description/urdf/bumperbot.urdf.xacro (robot description, xacro)
@@ -10,4 +10,7 @@
     <material name="YELLOW">
         <color rgba="1.0 1.0 0.0 1.0" /> <!-- rviz yellow color -->
+    </material>
+    <material name="RED">
+        <color rgba="1.0 0.0 0.0 1.0" /> <!-- rviz red color -->
     </material>
     <!--base_footprint
@@ -106,3 +109,21 @@
         <origin xyz="-0.04755 0.0 -0.0275" rpy="0.0 0.0 0.0" />
     </joint>
+    <!--can_link
+    link-->
+    <link name="can_link">
+        <visual>
+            <origin xyz="-0.032 0.032 0.0" rpy="${pi/2} 0.0 0.0" />
+            <geometry>
+                <mesh filename="package://bumperbot_description/meshes/can.STL" />
+            </geometry>
+            <material name="RED"/> <!-- color for rviz -->
+        </visual>
+    </link>
+    <!--base_joint
+    joint-->
+    <joint name="can_joint" type="fixed">
+        <parent link="base_link" />
+        <child link="can_link" />
+        <origin xyz="0.0 0.0 0.078" rpy="0.0 0.0 0.0" />
+    </joint>
 </robot>

Commit message: Add physical properties to URDF

File: src/bumperbot_description/urdf/bumperbot.urdf.xacro (robot description, xacro)
@@ -14,4 +14,5 @@
         <color rgba="1.0 0.0 0.0 1.0" /> <!-- rviz red color -->
     </material>
+    <xacro:include filename="$(find bumperbot_description)/urdf/bumperbot_gazebo.urdf" />
     <!--base_footprint
     link-->
@@ -20,4 +21,11 @@
     link-->
     <link name="base_link">
+        <inertial>
+            <origin xyz="0.0 0.0 0.04" rpy="0.0 0.25 0.3" />
+            <mass value="8.2573504e-01" />
+            <inertia ixx="2.2124416e-02" ixy="-1.2294101e-04" ixz="3.4938785e-04"
+                iyy="2.1193702e-02" iyz="-5.0120904e-05"
+                izz="2.0064271e-02" />
+        </inertial>
         <visual>
             <origin xyz="0.0 0.0 0.0" rpy="0.0 0.0 0.0" />
@@ -25,6 +33,12 @@
                 <mesh filename="package://bumperbot_description/meshes/base_link.STL" />
             </geometry>
-            <material name="WHITE"/> <!-- color for rviz -->
-        </visual>
+            <material name="WHITE" /> <!-- color for rviz -->
+        </visual>
+        <collision>
+            <origin xyz="0.0 0.0 0.0" rpy="0.0 0.0 0.0" />
+            <geometry>
+                <mesh filename="package://bumperbot_description/meshes/base_link.STL" />
+            </geometry>
+        </collision>
     </link>
     <!--base_joint
@@ -38,4 +52,12 @@
     link-->
     <link name="wheel_right_link">
+        <inertial>
+            <origin xyz="0 -0.014 0" rpy="0 0 0" />
+            <mass value="0.0530086090966721" />
+            <inertia ixx="1.88176298336665E-05" ixy="-4.8444933029987E-10"
+                ixz="1.88163708851143E-08"
+                iyy="3.11510738647764E-05" iyz="-6.93560663069607E-11"
+                izz="1.8801969558182E-05" />
+        </inertial>
         <visual>
             <origin xyz="0.0 0.0 0.0" rpy="${pi/2} 0.0 0.0" />
@@ -43,6 +65,12 @@
                 <mesh filename="package://bumperbot_description/meshes/wheel_right_link.STL" />
             </geometry>
-            <material name="CYAN"/> <!-- color for rviz -->
-        </visual>
+            <material name="CYAN" /> <!-- color for rviz -->
+        </visual>
+        <collision>
+            <origin xyz="0.0 -0.015 0.0" rpy="${pi/2} 0.0 0.0" />
+            <geometry>
+                <sphere radius="0.033" />
+            </geometry>
+        </collision>
     </link>
     <!--wheel_right_joint
@@ -57,4 +85,12 @@
     link-->
     <link name="wheel_left_link">
+        <inertial>
+            <origin xyz="0 0.014 0" rpy="0 0 0" />
+            <mass value="0.0530086043217644" />
+            <inertia ixx="1.8792911368909E-05" ixy="3.31256392204584E-10"
+                ixz="-1.14082001662767E-08"
+                iyy="3.11510738759073E-05" iyz="-3.60499245082192E-10"
+                izz="1.88266886146847E-05" />
+        </inertial>
         <visual>
             <origin xyz="0.0 0.0 0.0" rpy="${-pi/2} 0.0 0.0" />
@@ -62,6 +98,12 @@
                 <mesh filename="package://bumperbot_description/meshes/wheel_left_link.STL" />
             </geometry>
-            <material name="CYAN"/> <!-- color for rviz -->
-        </visual>
+            <material name="CYAN" /> <!-- color for rviz -->
+        </visual>
+        <collision>
+            <origin xyz="0.0 0.015 0.0" rpy="${-pi/2} 0.0 0.0" />
+            <geometry>
+                <sphere radius="0.033" />
+            </geometry>
+        </collision>
     </link>
     <!--wheel_left_joint
@@ -76,4 +118,12 @@
     link-->
     <link name="caster_front_link">
+        <inertial>
+            <origin xyz="3.89968128948481E-07 2.40073004698083E-07 0.00219173397061506" rpy="0 0 0" />
+            <mass value="1.44379265037903E-06" />
+            <inertia ixx="7.23075276010246E-11" ixy="-6.10956883467859E-16"
+                ixz="2.22849693525031E-15"
+                iyy="3.8713793085917E-11" iyz="2.93909858781952E-15"
+                izz="1.00967486676306E-10" />
+        </inertial>
         <visual>
             <origin xyz="0.0 0.0 0.0" rpy="0.0 0.0 0.0" />
@@ -81,6 +131,12 @@
                 <mesh filename="package://bumperbot_description/meshes/caster_front_link.STL" />
             </geometry>
-            <material name="YELLOW"/> <!-- color for rviz -->
-        </visual>
+            <material name="YELLOW" /> <!-- color for rviz -->
+        </visual>
+        <collision>
+            <origin xyz="0.0 0.0 0.0" rpy="0.0 0.0 0.0" />
+            <geometry>
+                <sphere radius="0.005" />
+            </geometry>
+        </collision>
     </link>
     <!--caster_front_joint
@@ -94,4 +150,13 @@
     link-->
     <link name="caster_rear_link">
+        <inertial>
+            <origin xyz="3.8996812895542E-07 2.40073004698083E-07 0.00219173397061509"
+                rpy="0 0 0" />
+            <mass value="1.44379265037902E-06" />
+            <inertia ixx="7.23075276010246E-11" ixy="-6.10956872363424E-16"
+                ixz="2.22849693527207E-15"
+                iyy="3.87137930859167E-11" iyz="2.939098587861E-15"
+                izz="1.00967486676306E-10" />
+        </inertial>
         <visual>
             <origin xyz="0.0 0.0 0.0" rpy="0.0 0.0 0.0" />
@@ -99,6 +164,12 @@
                 <mesh filename="package://bumperbot_description/meshes/caster_rear_link.STL" />
             </geometry>
-            <material name="YELLOW"/> <!-- color for rviz -->
-        </visual>
+            <material name="YELLOW" /> <!-- color for rviz -->
+        </visual>
+        <collision>
+            <origin xyz="0.0 0.0 0.0" rpy="0.0 0.0 0.0" />
+            <geometry>
+                <sphere radius="0.005" />
+            </geometry>
+        </collision>
     </link>
     <!--caster_rear_joint
@@ -117,5 +188,5 @@
                 <mesh filename="package://bumperbot_description/meshes/can.STL" />
             </geometry>
-            <material name="RED"/> <!-- color for rviz -->
+            <material name="RED" /> <!-- color for rviz -->
         </visual>
     </link>

Commit message: In URDF fix typo, and comment out the can from Assignment 1

File: src/bumperbot_description/urdf/bumperbot.urdf.xacro (robot description, xacro)
@@ -14,5 +14,5 @@
         <color rgba="1.0 0.0 0.0 1.0" /> <!-- rviz red color -->
     </material>
-    <xacro:include filename="$(find bumperbot_description)/urdf/bumperbot_gazebo.urdf" />
+    <xacro:include filename="$(find bumperbot_description)/urdf/bumperbot_gazebo.xacro" />
     <!--base_footprint
     link-->
@@ -180,6 +180,5 @@
         <origin xyz="-0.04755 0.0 -0.0275" rpy="0.0 0.0 0.0" />
     </joint>
-    <!--can_link
-    link-->
+    <!-- Assignment 1: add can on top of the robot
     <link name="can_link">
         <visual>
@@ -188,9 +187,7 @@
                 <mesh filename="package://bumperbot_description/meshes/can.STL" />
             </geometry>
-            <material name="RED" /> <!-- color for rviz -->
+            <material name="RED" />
         </visual>
     </link>
-    <!--base_joint
-    joint-->
     <joint name="can_joint" type="fixed">
         <parent link="base_link" />
@@ -198,3 +195,4 @@
         <origin xyz="0.0 0.0 0.078" rpy="0.0 0.0 0.0" />
     </joint>
+    -->
 </robot>

Commit message: Add ros2_control support to bumperbot - initial commit
 - modify bumperbot_gazebo.xacro to add transmission tags for joints and ros2_control plugin
 - create bumperbot_ros2_control.xacro to add a ros2_control tag with the gazebo plugin, and
   hardware interfaces for the joints
 - modify bumperbot.urdf.xacro to include bumperbot_ros2_control.xacro
 - create bumperbot_controller package and bumperbot_controllers.yaml configuration file
   with configuration for the controller_manager node
 - add notes in Section_5_Control

File: src/bumperbot_description/urdf/bumperbot.urdf.xacro (robot description, xacro)
@@ -1,5 +1,5 @@
 <?xml version="1.0"?>
 <robot xmlns:xacro="https://www.ros.org/wiki/xacro" name="bumperbot">
-    <!-- define color for rviz -->
+    <!-- define colors for rviz -->
     <material name="WHITE">
         <color rgba="1.0 1.0 1.0 1.0" /> <!-- rviz white color -->
@@ -14,10 +14,11 @@
         <color rgba="1.0 0.0 0.0 1.0" /> <!-- rviz red color -->
     </material>
+    <!-- include gazebo xacro file -->
     <xacro:include filename="$(find bumperbot_description)/urdf/bumperbot_gazebo.xacro" />
-    <!--base_footprint
-    link-->
+    <!-- include ros2 control xacro file -->
+    <xacro:include filename="$(find bumperbot_description)/urdf/bumperbot_ros2_control.xacro"/>
+    <!-- base_footprint link -->
     <link name="base_footprint" />
-    <!--base_link
-    link-->
+    <!-- base_link link -->
     <link name="base_link">
         <inertial>
@@ -42,6 +43,5 @@
         </collision>
     </link>
-    <!--base_joint
-    joint-->
+    <!-- base_joint joint -->
     <joint name="base_joint" type="fixed">
         <parent link="base_footprint" />
@@ -49,6 +49,5 @@
         <origin xyz="0.0 0.0 0.033" rpy="0.0 0.0 0.0" />
     </joint>
-    <!--wheel_right_link
-    link-->
+    <!-- wheel_right_link link -->
     <link name="wheel_right_link">
         <inertial>
@@ -74,6 +73,5 @@
         </collision>
     </link>
-    <!--wheel_right_joint
-    joint-->
+    <!-- wheel_right_joint joint -->
     <joint name="wheel_right_joint" type="continuous">
         <parent link="base_link" />
@@ -82,6 +80,5 @@
         <origin xyz="0.0 -0.07 0.0" rpy="0.0 0.0 0.0" />
     </joint>
-    <!--wheel_left_link
-    link-->
+    <!-- wheel_left_link link -->
     <link name="wheel_left_link">
         <inertial>
@@ -107,6 +104,5 @@
         </collision>
     </link>
-    <!--wheel_left_joint
-    joint-->
+    <!-- wheel_left_joint joint -->
     <joint name="wheel_left_joint" type="continuous">
         <parent link="base_link" />
@@ -115,6 +111,5 @@
         <origin xyz="0.0 0.07 0.0" rpy="0.0 0.0 0.0" />
     </joint>
-    <!--caster_front_link
-    link-->
+    <!-- caster_front_link link-->
     <link name="caster_front_link">
         <inertial>
@@ -140,6 +135,5 @@
         </collision>
     </link>
-    <!--caster_front_joint
-    joint-->
+    <!-- caster_front_joint joint-->
     <joint name="caster_front_joint" type="fixed">
         <parent link="base_link" />
@@ -147,6 +141,5 @@
         <origin xyz="0.04755 0.0 -0.0275" rpy="0.0 0.0 0.0" />
     </joint>
-    <!--caster_rear_link
-    link-->
+    <!-- caster_rear_link link -->
     <link name="caster_rear_link">
         <inertial>
@@ -173,6 +166,5 @@
         </collision>
     </link>
-    <!--caster_rear_joint
-    joint-->
+    <!-- caster_rear_joint joint -->
     <joint name="caster_rear_joint" type="fixed">
         <parent link="base_link" />

File: src/bumperbot_description/urdf/bumperbot_gazebo.xacro (robot description, xacro)
@@ -1,4 +1,20 @@
 <?xml version="1.0"?>
 <robot xmlns:xacro="https://www.ros.org/wiki/xacro" name="bumperbot">
+<!-- wheel right transmission -->
+ <transmission name="wheel_right_transmission">
+    <plugin>transmission_interface/SimpleTransmission</plugin>
+    <actuator name="wheel_right_motor" role="actuator_right"/>
+    <joint name="wheel_right_joint" role="joint_right">
+        <mechanical_reduction>1.0</mechanical_reduction>
+    </joint>
+</transmission>
+<!-- wheel left transmission -->
+<transmission name="wheel_left_transmission">
+    <plugin>transmission_interface/SimpleTransmission</plugin>
+    <actuator name="wheel_left_motor" role="actuator_left"/>
+    <joint name="wheel_left_joint" role="joint_left">
+        <mechanical_reduction>1.0</mechanical_reduction>
+    </joint>
+</transmission>
 <gazebo reference="wheel_right_link">
     <!-- friction coefficients -->
@@ -39,3 +55,13 @@
     <maxVel>0.1</maxVel>
 </gazebo>
+<!-- ros2 control library support -->
+<gazebo>
+    <plugin filename="libgazebo_ros2_control.so" name="gazebo_ros2_control">
+        <robot_param>robot_description</robot_param> <!-- topic -->
+        <robot_param_node>robot_state_publisher</robot_param_node> <!-- publisher node -->
+        <parameters>
+            $(find bumperbot_controller)/config/bumperbot_controllers.yaml
+        </parameters>
+    </plugin>
+</gazebo>
 </robot>
